File: eagle-cad/ppm-converter.sch (EAGLE design)
At the start: 18 parts, among them IC1 74HC14, IC2 74HC14, U1 ATMEGA328P, Y1 16Mhz

Commit message: Added ISP-header
Parts:
- added ISP: (no value), SparkFun-Connectors:M06SIP
Connections:
- new net N$18: ISP.1, U1.PB4(MISO)
- new net N$28: ISP.3, U1.PB5(SCK)
- new net N$29: ISP.4, U1.PB3(MOSI/OC2)
- net GND: now also ISP.6
- net N$4: now also ISP.5
- net VCC: now also ISP.2
Changed lines of the file:
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@@
 <?xml version="1.0" encoding="utf-8"?>
 <!DOCTYPE eagle SYSTEM "eagle.dtd">
-<eagle version="6.3">
+<eagle version="6.4">
 <drawing>
 <settings>
@@
 <part name="P+5" library="SparkFun-Aesthetics" deviceset="VCC" device=""/>
 <part name="P+6" library="SparkFun-Aesthetics" deviceset="VCC" device=""/>
+<part name="ISP" library="SparkFun-Connectors" deviceset="M06" device="SIP"/>
+<part name="P+7" library="SparkFun-Aesthetics" deviceset="VCC" device=""/>
+<part name="GND11" library="SparkFun-Aesthetics" deviceset="GND" device=""/>
 </parts>
 <sheets>
@@
 <instance part="P+5" gate="1" x="83.82" y="48.26"/>
 <instance part="P+6" gate="1" x="121.92" y="96.52"/>
+<instance part="ISP" gate="G$1" x="2.54" y="139.7"/>
+<instance part="P+7" gate="1" x="12.7" y="149.86"/>
+<instance part="GND11" gate="1" x="10.16" y="152.4" rot="R180"/>
 </instances>
 <busses>
@@
 <wire x1="81.28" y1="149.86" x2="81.28" y2="147.32" width="0.1524" layer="91"/>
 </segment>
+<segment>
+<pinref part="ISP" gate="G$1" pin="6"/>
+<wire x1="7.62" y1="147.32" x2="10.16" y2="147.32" width="0.1524" layer="91"/>
+<pinref part="GND11" gate="1" pin="GND"/>
+<wire x1="10.16" y1="147.32" x2="10.16" y2="149.86" width="0.1524" layer="91"/>
+</segment>
 </net>
 <net name="N$4" class="0">
@@
 <pinref part="R1" gate="G$1" pin="1"/>
 <wire x1="104.14" y1="78.74" x2="106.68" y2="78.74" width="0.1524" layer="91"/>
+<wire x1="106.68" y1="78.74" x2="106.68" y2="73.66" width="0.1524" layer="91"/>
+<wire x1="106.68" y1="73.66" x2="43.18" y2="73.66" width="0.1524" layer="91"/>
+<wire x1="43.18" y1="73.66" x2="43.18" y2="144.78" width="0.1524" layer="91"/>
+<pinref part="ISP" gate="G$1" pin="5"/>
+<wire x1="43.18" y1="144.78" x2="7.62" y2="144.78" width="0.1524" layer="91"/>
+<junction x="106.68" y="78.74"/>
 </segment>
 </net>
@@
 <pinref part="P+6" gate="1" pin="VCC"/>
 </segment>
+<segment>
+<pinref part="ISP" gate="G$1" pin="2"/>
+<wire x1="7.62" y1="137.16" x2="12.7" y2="137.16" width="0.1524" layer="91"/>
+<pinref part="P+7" gate="1" pin="VCC"/>
+<wire x1="12.7" y1="137.16" x2="12.7" y2="149.86" width="0.1524" layer="91"/>
+</segment>
 </net>
 <net name="N$1" class="0">
@@
 </segment>
 </net>
+<net name="N$18" class="0">
+<segment>
+<pinref part="U1" gate="G$1" pin="PB4(MISO)"/>
+<wire x1="55.88" y1="134.62" x2="7.62" y2="134.62" width="0.1524" layer="91"/>
+<pinref part="ISP" gate="G$1" pin="1"/>
+</segment>
+</net>
+<net name="N$28" class="0">
+<segment>
+<pinref part="U1" gate="G$1" pin="PB5(SCK)"/>
+<wire x1="55.88" y1="137.16" x2="15.24" y2="137.16" width="0.1524" layer="91"/>
+<wire x1="15.24" y1="137.16" x2="15.24" y2="139.7" width="0.1524" layer="91"/>
+<pinref part="ISP" gate="G$1" pin="3"/>
+<wire x1="15.24" y1="139.7" x2="7.62" y2="139.7" width="0.1524" layer="91"/>
+</segment>
+</net>
+<net name="N$29" class="0">
+<segment>
+<pinref part="U1" gate="G$1" pin="PB3(MOSI/OC2)"/>
+<wire x1="55.88" y1="132.08" x2="17.78" y2="132.08" width="0.1524" layer="91"/>
+<wire x1="17.78" y1="132.08" x2="17.78" y2="142.24" width="0.1524" layer="91"/>
+<pinref part="ISP" gate="G$1" pin="4"/>
+<wire x1="17.78" y1="142.24" x2="7.62" y2="142.24" width="0.1524" layer="91"/>
+</segment>
+</net>

Commit message: Added led+resistor, finetuning some titles
Parts:
- added LED: (no value), SparkFun-LED:LED5MM-KIT
- added R3: LED, SparkFun-Passives:RESISTORAXIAL-0.3
Connections:
- new net N$21: LED.A, R3.1
- new net N$31: R3.2, U1.PC0(ADC0)
- net GND: now also LED.C
Changed lines of the file:
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@@
 <part name="P+7" library="SparkFun-Aesthetics" deviceset="VCC" device=""/>
 <part name="GND11" library="SparkFun-Aesthetics" deviceset="GND" device=""/>
+<part name="LED" library="SparkFun-LED" deviceset="LED" device="5MM-KIT"/>
+<part name="GND12" library="SparkFun-Aesthetics" deviceset="GND" device=""/>
+<part name="R3" library="SparkFun-Passives" deviceset="RESISTOR" device="AXIAL-0.3" value="LED"/>
 </parts>
 <sheets>
@@
 <instance part="P+7" gate="1" x="12.7" y="149.86"/>
 <instance part="GND11" gate="1" x="10.16" y="152.4" rot="R180"/>
+<instance part="LED" gate="G$1" x="35.56" y="40.64"/>
+<instance part="GND12" gate="1" x="35.56" y="30.48"/>
+<instance part="R3" gate="G$1" x="35.56" y="50.8" rot="R90"/>
 </instances>
 <busses>
@@
 <pinref part="GND11" gate="1" pin="GND"/>
 <wire x1="10.16" y1="147.32" x2="10.16" y2="149.86" width="0.1524" layer="91"/>
+</segment>
+<segment>
+<pinref part="LED" gate="G$1" pin="C"/>
+<pinref part="GND12" gate="1" pin="GND"/>
+<wire x1="35.56" y1="35.56" x2="35.56" y2="33.02" width="0.1524" layer="91"/>
 </segment>
 </net>
@@
 </segment>
 </net>
+<net name="N$21" class="0">
+<segment>
+<pinref part="R3" gate="G$1" pin="1"/>
+<pinref part="LED" gate="G$1" pin="A"/>
+<wire x1="35.56" y1="45.72" x2="35.56" y2="43.18" width="0.1524" layer="91"/>
+</segment>
+</net>
+<net name="N$31" class="0">
+<segment>
+<pinref part="U1" gate="G$1" pin="PC0(ADC0)"/>
+<pinref part="R3" gate="G$1" pin="2"/>
+<wire x1="55.88" y1="78.74" x2="35.56" y2="78.74" width="0.1524" layer="91"/>
+<wire x1="35.56" y1="78.74" x2="35.56" y2="55.88" width="0.1524" layer="91"/>
+</segment>
+</net>

Commit message: Changed version -> revision, added 0.1uF cap
Parts:
- added C5: 0.1uF, SparkFun-Passives:CAPPTH
Connections:
- net GND: now also C5.2
- net VCC: now also C5.1
Changed lines of the file:
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@@
 <part name="GND12" library="SparkFun-Aesthetics" deviceset="GND" device=""/>
 <part name="R3" library="SparkFun-Passives" deviceset="RESISTOR" device="AXIAL-0.3" value="LED"/>
+<part name="C5" library="SparkFun-Passives" deviceset="CAP" device="PTH" value="0.1uF"/>
 </parts>
 <sheets>
@@
 <instance part="GND12" gate="1" x="35.56" y="30.48"/>
 <instance part="R3" gate="G$1" x="35.56" y="50.8" rot="R90"/>
+<instance part="C5" gate="G$1" x="132.08" y="76.2"/>
 </instances>
 <busses>
@@
 <wire x1="127" y1="71.12" x2="121.92" y2="71.12" width="0.1524" layer="91"/>
 <junction x="121.92" y="71.12"/>
+<wire x1="127" y1="71.12" x2="132.08" y2="71.12" width="0.1524" layer="91"/>
+<pinref part="C5" gate="G$1" pin="2"/>
+<wire x1="132.08" y1="71.12" x2="132.08" y2="73.66" width="0.1524" layer="91"/>
+<junction x="127" y="71.12"/>
 </segment>
 <segment>
@@
 <junction x="116.84" y="83.82"/>
 <pinref part="P+6" gate="1" pin="VCC"/>
-</segment>
-<segment>
+<pinref part="C5" gate="G$1" pin="1"/>
+<wire x1="127" y1="83.82" x2="132.08" y2="83.82" width="0.1524" layer="91"/>
+<wire x1="132.08" y1="83.82" x2="132.08" y2="81.28" width="0.1524" layer="91"/>
+<junction x="127" y="83.82"/>
+</segment>
+<segment>
